File: Controller/SOC_Power.kicad_sch (KiCad schematic)
At the start: 80 parts, among them U11 AM6252ASGFHIAMCRQ1

Commit message: Fixed some minor issues, started some scheamtic clean up
Parts:
- C100, C103, C22, C23, C24, C25, C26, C27, C32, C33, C34, C35, C36, C39, C40, C41, C47, C49, C50, C51, C52, C64, C65, C66, C67, C68, C84: now not fitted
Changed lines of the file:
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@@
 		(exclude_from_sim no)
 		(in_bom yes)
-		(on_board yes)
-		(dnp no)
+		(on_board no)
+		(dnp yes)
 		(property "Reference" "C32"
 			(at 194.31 265.4299 0)
@@
 		(exclude_from_sim no)
 		(in_bom yes)
-		(on_board yes)
-		(dnp no)
+		(on_board no)
+		(dnp yes)
 		(property "Reference" "C27"
 			(at 130.81 265.4299 0)
@@
 		(exclude_from_sim no)
 		(in_bom yes)
-		(on_board yes)
-		(dnp no)
+		(on_board no)
+		(dnp yes)
 		(property "Reference" "C103"
 			(at 214.63 97.79 0)
@@
 		(exclude_from_sim no)
 		(in_bom yes)
-		(on_board yes)
-		(dnp no)
+		(on_board no)
+		(dnp yes)
 		(property "Reference" "C34"
 			(at 219.71 265.4299 0)
@@
 		(exclude_from_sim no)
 		(in_bom yes)
-		(on_board yes)
-		(dnp no)
+		(on_board no)
+		(dnp yes)
 		(property "Reference" "C52"
 			(at 118.11 241.2999 0)
@@
 		(exclude_from_sim no)
 		(in_bom yes)
-		(on_board yes)
-		(dnp no)
+		(on_board no)
+		(dnp yes)
 		(property "Reference" "C41"
 			(at 245.11 241.2999 0)
@@
 		(exclude_from_sim no)
 		(in_bom yes)
-		(on_board yes)
-		(dnp no)
+		(on_board no)
+		(dnp yes)
 		(property "Reference" "C66"
 			(at 231.14 218.4399 0)
@@
 		(exclude_from_sim no)
 		(in_bom yes)
-		(on_board yes)
-		(dnp no)
+		(on_board no)
+		(dnp yes)
 		(property "Reference" "C65"
 			(at 218.44 218.4399 0)
@@
 		(exclude_from_sim no)
 		(in_bom yes)
-		(on_board yes)
-		(dnp no)
+		(on_board no)
+		(dnp yes)
 		(property "Reference" "C51"
 			(at 105.41 241.2999 0)
@@
 		(exclude_from_sim no)
 		(in_bom yes)
-		(on_board yes)
-		(dnp no)
+		(on_board no)
+		(dnp yes)
 		(property "Reference" "C26"
 			(at 118.11 265.4299 0)
@@
 		(exclude_from_sim no)
 		(in_bom yes)
-		(on_board yes)
-		(dnp no)
+		(on_board no)
+		(dnp yes)
 		(property "Reference" "C50"
 			(at 92.71 241.2999 0)
@@
 		(exclude_from_sim no)
 		(in_bom yes)
-		(on_board yes)
-		(dnp no)
+		(on_board no)
+		(dnp yes)
 		(property "Reference" "C24"
 			(at 92.71 265.4299 0)
@@
 		(exclude_from_sim no)
 		(in_bom yes)
-		(on_board yes)
-		(dnp no)
+		(on_board no)
+		(dnp yes)
 		(property "Reference" "C47"
 			(at 64.77 241.3 0)
@@
 		(exclude_from_sim no)
 		(in_bom yes)
-		(on_board yes)
-		(dnp no)
+		(on_board no)
+		(dnp yes)
 		(property "Reference" "C22"
 			(at 64.77 265.43 0)
@@
 		(exclude_from_sim no)
 		(in_bom yes)
-		(on_board yes)
-		(dnp no)
+		(on_board no)
+		(dnp yes)
 		(property "Reference" "C67"
 			(at 243.84 218.4399 0)
@@
 		(exclude_from_sim no)
 		(in_bom yes)
-		(on_board yes)
-		(dnp no)
+		(on_board no)
+		(dnp yes)
 		(property "Reference" "C39"
 			(at 219.71 241.2999 0)
@@
 		(exclude_from_sim no)
 		(in_bom yes)
-		(on_board yes)
-		(dnp no)
+		(on_board no)
+		(dnp yes)
 		(property "Reference" "C84"
 			(at 214.63 48.26 0)
@@
 		(exclude_from_sim no)
 		(in_bom yes)
-		(on_board yes)
-		(dnp no)
+		(on_board no)
+		(dnp yes)
 		(property "Reference" "C100"
 			(at 214.63 72.39 0)
@@
 		(exclude_from_sim no)
 		(in_bom yes)
-		(on_board yes)
-		(dnp no)
+		(on_board no)
+		(dnp yes)
 		(property "Reference" "C40"
 			(at 232.41 241.2999 0)
@@
 		(exclude_from_sim no)
 		(in_bom yes)
-		(on_board yes)
-		(dnp no)
+		(on_board no)
+		(dnp yes)
 		(property "Reference" "C35"
 			(at 232.41 265.4299 0)
@@
 		(exclude_from_sim no)
 		(in_bom yes)
-		(on_board yes)
-		(dnp no)
+		(on_board no)
+		(dnp yes)
 		(property "Reference" "C64"
 			(at 205.74 218.4399 0)
@@
 		(exclude_from_sim no)
 		(in_bom yes)
-		(on_board yes)
-		(dnp no)
+		(on_board no)
+		(dnp yes)
 		(property "Reference" "C33"
 			(at 207.01 265.4299 0)
@@
 	(symbol
 		(lib_id "power:VCC")
-		(at 172.72 132.08 0)
-		(unit 1)
-		(exclude_from_sim no)
-		(in_bom yes)
-		(on_board yes)
-		(dnp no)
-		(fields_autoplaced yes)
-		(property "Reference" "#PWR0589"
-			(at 172.72 135.89 0)
-			(effects
-				(font
-					(size 1.27 1.27)
-				)
-				(hide yes)
-			)
-		)
-		(property "Value" "VDD_SDIO"
-			(at 175.26 130.8099 0)
-			(effects
-				(font
-					(size 1.27 1.27)
-				)
-				(justify left)
-			)
-		)
-		(property "Footprint" ""
-			(at 172.72 132.08 0)
-			(effects
-				(font
-					(size 1.27 1.27)
-				)
-				(hide yes)
-			)
-		)
-		(property "Datasheet" ""
-			(at 172.72 132.08 0)
-			(effects
-				(font
-					(size 1.27 1.27)
-				)
-				(hide yes)
-			)
-		)
-		(property "Description" "Power symbol creates a global label with name \"VCC\""
-			(at 172.72 132.08 0)
-			(effects
-				(font
-					(size 1.27 1.27)
-				)
-				(hide yes)
-			)
-		)
-		(pin "1"
-		)
-		(instances
-			(project "Controller"
-				(path "/2c9e7a41-63e4-4339-89dd-991e772f7a19/25cc9d1f-4661-44d6-b5ea-319405d0978d"
-					(reference "#PWR0589")
-					(unit 1)
-				)
-			)
-		)
-	)
-	(symbol
-		(lib_id "power:VCC")
 		(at 172.72 68.58 0)
 		(unit 1)
@@
 		(exclude_from_sim no)
 		(in_bom yes)
-		(on_board yes)
-		(dnp no)
+		(on_board no)
+		(dnp yes)
 		(property "Reference" "C23"
 			(at 80.01 265.4299 0)
@@
 		(exclude_from_sim no)
 		(in_bom yes)
-		(on_board yes)
-		(dnp no)
+		(on_board no)
+		(dnp yes)
 		(property "Reference" "C25"
 			(at 105.41 265.4299 0)
@@
 		(exclude_from_sim no)
 		(in_bom yes)
-		(on_board yes)
-		(dnp no)
+		(on_board no)
+		(dnp yes)
 		(property "Reference" "C49"
 			(at 80.01 241.2999 0)
@@
 		(exclude_from_sim no)
 		(in_bom yes)
-		(on_board yes)
-		(dnp no)
+		(on_board no)
+		(dnp yes)
 		(property "Reference" "C68"
 			(at 256.54 218.4399 0)
@@
 		(exclude_from_sim no)
 		(in_bom yes)
-		(on_board yes)
-		(dnp no)
+		(on_board no)
+		(dnp yes)
 		(property "Reference" "C36"
 			(at 245.11 265.4299 0)
