File: Controller/ADC.kicad_sch (KiCad schematic)
At the start: 51 parts, among them J11 Conn_01x02_Socket, J12 Conn_01x02_Socket, J22 Conn_01x02_Socket, J23 Conn_01x02_Socket, J28 Conn_01x04_Socket, J29 Conn_01x04_Socket, SW2 SW_DIP_x04, U29 ADS124S08IPBSR, U37 TLV75533PDBV

Commit message: Testpoints + DDR velocity comp
Parts:
- added R179: 10K, Resistor_SMD:R_0603_1608Metric, symbol Device:R
Connections:
- net +3V3_SYS: now also R179.2
- net +5V: no longer U37.3 (EN)
- new net: R179.1, U37.3 (EN)
Other:
- note added: "TODO: RREF will need to be adjusted"
- note removed: "Need to replace footprint"
- note removed: "TODO: RREF will need to be adjusted properly"
- moved on the sheet: C302
