File: Controller/Heaters.kicad_sch (KiCad schematic)
At the start: 33 parts, among them J21 Screw_Terminal_01x06, Q5 IRFB7440PBF, Q6 HYG009N04LS1C2, Q7 HYG009N04LS1C2, Q8 HYG009N04LS1C2, U20 UCC27524DR, U21 UCC27524DR

Commit message: Testpoints + DDR velocity comp
Parts:
- added TP28, TP29, TP30, TP31: TestPoint, TestPoint:TestPoint_Pad_D1.5mm, symbol Connector:TestPoint
Connections:
- net H0_PWM: now also TP28.1
- net H1_PWM: now also TP31.1
- net H2_PWM: now also TP30.1
- net HBED_PWM: now also TP29.1
Other:
- moved on the sheet: C198, C199, D16, D17, D18, D19, D20, D21, D22, D23, J21, Q5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
