File: Controller/M.2_KeyE_WIFI.kicad_sch (KiCad schematic)
At the start: 23 parts, among them J54 MDT275E01001, U42 SN74LVC1T45DBV, U43 SN74LVC1T45DBV, U44 SN74LVC1T45DBV, U45 SN74LVC1T45DBV

Commit message: Testpoints + DDR velocity comp
Parts:
- removed R179: 10K, Resistor_SMD:R_0603_1608Metric, symbol Device:R
- added R232, R233: 10K, Resistor_SMD:R_0603_1608Metric, symbol Device:R
- added TP18, TP19, TP20: TestPoint, TestPoint:TestPoint_Pad_D1.0mm, symbol Connector:TestPoint
Connections:
- net BT_UART_WAKE: now also R232.1, TP19.1
- net GND: now also R232.2, R233.2
- net MMC2_SDCD: now also TP18.1
- net MMC2_SDWP: now also TP20.1
- net WlAN_EN: now also R233.1
