File: Controller/MMC.kicad_sch (KiCad schematic)
At the start: 42 parts, among them J44 Micro_SD_Card_Det1, U11 AM6252ASGFHIAMCRQ1, U23 74LVC1G08, U31 TPS22918DBV, U32 74LVC1G08, U36 EMMC08G-MB29-PM9B

Commit message: JTAG
Parts:
- removed C82: 1000pF 12kV, Capacitor_SMD:C_1206_3216Metric, symbol Device:C
Connections:
- net Earth is gone; now on net GND: J44.10 (SHIELD)

Commit message: Testpoints + DDR velocity comp
Parts:
- added R234: 10K, Resistor_SMD:R_0603_1608Metric, symbol Device:R
- added TP23, TP24: TestPoint, TestPoint:TestPoint_Pad_D1.5mm, symbol Connector:TestPoint
Connections:
- net +3V3_SYS: now also R234.1
- net EMMC1_RST: now also R234.2, TP24.1
- net EMMC_~{RST}: now also TP23.1
