File: Controller/SOC_USB.kicad_sch (KiCad schematic)
At the start: 48 parts, among them J1 USB_A_Stacked, J3 USB_A_Stacked, J53 USB_A, U11 AM6252ASGFHIAMCRQ1, U12 USB2514B-AEZC-TR, U16 TPD3S014, U17 TPD3S014, U18 TPD3S014, U19 TPD3S014, U34 TPD3S044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

Commit message: Testpoints + DDR velocity comp
Parts:
- added TP25, TP26: TestPoint, TestPoint:TestPoint_Pad_D1.5mm, symbol Connector:TestPoint
- added TP27: TestPoint, TestPoint:TestPoint_Pad_D1.0mm, symbol Connector:TestPoint
Connections:
- net USB0__DRVVBUS: now also TP25.1
- net USB1__DRVVBUS: now also TP27.1
- net at U12.12 (PRTPWR1), U16.1 (EN): now also TP26.1
