File: Controller/GPMC_Interface.kicad_sch (KiCad schematic)
At the start: 35 parts, among them SW1 SW_DIP_x04, SW3 SW_Push, SW4 SW_Push, U11 AM6252ASGFHIAMCRQ1

Commit message: DDR_CLK termination
Parts:
- added J61: TC2050, Connector:Tag-Connect_TC2050-IDC-NL_2x05_P1.27mm_Vertical, symbol Connector:TC2050
- added TP5: TestPoint, TestPoint:TestPoint_THTPad_D2.0mm_Drill1.0mm, symbol Connector:TestPoint
Connections:
- net TRSTN: now reaches U11.A11 (TRSTN)
- net TMS: now reaches U11.B11 (TMS)
- net TCK: now reaches U11.C10 (TCK)
- net TDI: now reaches U11.D10 (TDI)
- net TDO: now reaches U11.E10 (TDO)
- net UART0_TXD: now reaches R206.2, U11.E11 (UART0_TXD)
- net UART0_TXD: now also TP5.1
- net EMU1: now reaches U11.B10 (EMU1)
- net EMU0: now reaches U11.D9 (EMU0)
Other:
- note added: "JTAG"
- moved on the sheet: R206, R219, R220, SW3, SW4

Commit message: JTAG
Parts:
- added R226, R8, R9: 4K7, Resistor_SMD:R_0603_1608Metric, symbol Device:R
- added R227, R228, R229, R230: 10K, Resistor_SMD:R_0603_1608Metric, symbol Device:R
- added R231: 22R, Resistor_SMD:R_0402_1005Metric, symbol Device:R
Connections:
- net +3V3_SYS: now also J61.7, R226.1, R227.1, R228.1, R229.1, R8.1, R9.1
- net EMU0: now also J61.9, R228.2
- net EMU1: now also J61.10, R229.2
- net GND: now also J61.4, J61.6, R230.2
- net TCK: now also R231.1
- net TDI: now also J61.1, R8.2
- net TDO: now also J61.8, R227.2
- net TMS: now also J61.3, R226.2
- net TRSTN: now also J61.2, R9.2
- net at J61.5: now also R230.1, R231.2
Other:
- moved on the sheet: J61

Commit message: REV 1B
Parts:
- added TP35: TestPoint, TestPoint:TestPoint_Pad_D1.5mm, symbol Connector:TestPoint
Connections:
- net MCU__ERRORN: now reaches U11.B1 (MCU__ERRORN)
- net MCU__ERRORN: now also TP35.1
- net PMIC_INT_N: now reaches U11.B16 (EXTINTN)
- net PRU0_GPO10 renamed HDMI_INT
- no-connect marks 31 -> 30
Changed lines of the file:
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@@
 	)
 	(no_connect
-		(at 287.02 27.94)
-	)
-	(no_connect
 		(at 287.02 109.22)
 	)
@@
 	(wire
 		(pts
+			(xy 267.97 27.94) (xy 267.97 25.4)
+		)
+		(stroke
+			(width 0)
+			(type default)
+		)
+	)
+	(wire
+		(pts
 			(xy 146.05 107.95) (xy 146.05 101.6)
 		)
@@
 	(wire
 		(pts
+			(xy 267.97 27.94) (xy 287.02 27.94)
+		)
+		(stroke
+			(width 0)
+			(type default)
+		)
+	)
+	(wire
+		(pts
 			(xy 200.66 35.56) (xy 200.66 38.1)
 		)
@@
 	(wire
 		(pts
+			(xy 85.09 39.37) (xy 80.01 39.37)
+		)
+		(stroke
+			(width 0)
+			(type default)
+		)
+	)
+	(wire
+		(pts
 			(xy 373.38 80.01) (xy 368.3 80.01)
 		)
@@
 		)
 	)
+	(label "MCU__ERRORN"
+		(at 271.78 27.94 0)
+		(effects
+			(font
+				(size 1.27 1.27)
+			)
+			(justify left bottom)
+		)
+	)
 	(label "BOOTMODE_5"
 		(at 153.67 25.4 0)
@@
 		)
 	)
-	(global_label "PRU0_GPO10"
-		(shape input)
-		(at 85.09 115.57 0)
-		(fields_autoplaced yes)
-		(effects
-			(font
-				(size 1.27 1.27)
-			)
-			(justify left)
-		)
-		(property "Intersheetrefs" "${INTERSHEET_REFS}"
-			(at 100.4123 115.57 0)
-			(hide yes)
-			(show_name no)
-			(do_not_autoplace no)
-			(effects
-				(font
-					(size 1.27 1.27)
-				)
-				(justify left)
-			)
-		)
-	)
 	(global_label "VOUT0__DATA19"
 		(shape input)
@@
 		)
 	)
+	(global_label "PMIC_INT_N"
+		(shape input)
+		(at 85.09 39.37 0)
+		(fields_autoplaced yes)
+		(effects
+			(font
+				(size 1.27 1.27)
+			)
+			(justify left)
+		)
+		(property "Intersheetrefs" "${INTERSHEET_REFS}"
+			(at 98.84 39.37 0)
+			(hide yes)
+			(show_name no)
+			(do_not_autoplace no)
+			(effects
+				(font
+					(size 1.27 1.27)
+				)
+				(justify left)
+			)
+		)
+	)
 	(global_label "MCU_GPIO_1"
 		(shape input)
@@
 		)
 	)
+	(global_label "HDMI_INT"
+		(shape input)
+		(at 85.09 115.57 0)
+		(fields_autoplaced yes)
+		(effects
+			(font
+				(size 1.27 1.27)
+			)
+			(justify left)
+		)
+		(property "Intersheetrefs" "${INTERSHEET_REFS}"
+			(at 96.6024 115.57 0)
+			(hide yes)
+			(show_name no)
+			(do_not_autoplace no)
+			(effects
+				(font
+					(size 1.27 1.27)
+				)
+				(justify left)
+			)
+		)
+	)
 	(global_label "EHRPWM1_B"
 		(shape input)
@@
 					(unit 1)
 				)
+			)
+		)
+	)
+	(symbol
+		(lib_id "Connector:TestPoint")
+		(at 267.97 25.4 0)
+		(unit 1)
+		(body_style 1)
+		(exclude_from_sim no)
+		(in_bom yes)
+		(on_board yes)
+		(in_pos_files yes)
+		(dnp no)
+		(fields_autoplaced yes)
+		(property "Reference" "TP35"
+			(at 270.51 20.8279 0)
+			(show_name no)
+			(do_not_autoplace no)
+			(effects
+				(font
+					(size 1.27 1.27)
+				)
+				(justify left)
+			)
+		)
+		(property "Value" "TestPoint"
+			(at 270.51 23.3679 0)
+			(show_name no)
+			(do_not_autoplace no)
+			(effects
+				(font
+					(size 1.27 1.27)
+				)
+				(justify left)
+			)
+		)
+		(property "Footprint" "TestPoint:TestPoint_Pad_D1.5mm"
+			(at 273.05 25.4 0)
+			(hide yes)
+			(show_name no)
+			(do_not_autoplace no)
+			(effects
+				(font
+					(size 1.27 1.27)
+				)
+			)
+		)
+		(property "Datasheet" ""
+			(at 273.05 25.4 0)
+			(hide yes)
+			(show_name no)
+			(do_not_autoplace no)
+			(effects
+				(font
+					(size 1.27 1.27)
+				)
+			)
+		)
+		(property "Description" "test point"
+			(at 267.97 25.4 0)
+			(hide yes)
+			(show_name no)
+			(do_not_autoplace no)
+			(effects
+				(font
+					(size 1.27 1.27)
+				)
+			)
+		)
+		(pin "1"
+		)
+		(instances
+			(project "Controller"
+				(path "/2c9e7a41-63e4-4339-89dd-991e772f7a19/4f9a8529-8434-4a63-acea-238523d9a9d8"
+					(reference "TP35")
+					(unit 1)
+				)
